File: modules/cellular-modem/cellular-modem.kicad_pcb (KiCad board)
At the start: 2 copper layers, 42.8 x 71.1 mm, 23 parts, among them J1 MM60-52B1-E1-R650, J2 MM60-EZH059-B5-R650, U1 TXV0108RGYR, U2 TXV0108RGYR, U3 TXV0108RGYR, U4 TPS631000DRLR, U5 TPS631000DRLR

Commit message: Updating cellular modem - adding KiCad git ignore
Parts:
- J1: value MM60-52B1-E1-R650 -> MM60-mini-PCIe
- M1: footprint MegaCastle:MegaCastle2x28-Module-I36.0x66.3-MB00007FFFFFFFF-NIBBLE -> MegaCastle:MegaCastle2x28-Module-I42.8x66.3-MB00007FFFFFFFF-SPAREPAD
- U1, U2, U3: footprint footprints:VQFN24_RGY_TEX -> cellular-modem:VQFN24_RGY_TEX
Routing:
- net GND: track 129.0 -> 144.8 mm, vias 37 -> 113
- net 1V8: track 99.4 -> 95.1 mm
- net UART_TX_3V3: track 30.3 -> 32.7 mm
- net EN: track 61.9 -> 59.9 mm
- net Net-(JP1-A): track 12.4 -> 14.3 mm
- net //WAKE_OC_OUT: track 30.8 -> 32.5 mm
- net COEX_UART_TX_3V3: track 28.7 -> 30.3 mm
- net PETp0: track 20.3 -> 18.9 mm
- net /COEX_UART_RX_1V8_IN: track 22.0 -> 20.9 mm
- net /WAKE_3V3: track 27.2 -> 28.3 mm
- net /PCM_SYNC_1V8_IO: track 37.2 -> 38.2 mm
- net /PCM_DIN_1V8_IN: track 35.3 -> 36.1 mm
- net /COEX_UART_TX_1V8_OUT: track 28.7 -> 29.4 mm
- net RI_HOST_WAKE_3V3: track 25.6 -> 26.3 mm
- net /PCM_DOUT_1V8_OUT: track 29.1 -> 29.7 mm
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- added copper zone on In1.Cu, net GND
- added copper zone on In2.Cu, net GND
Other:
- outline, holes or cut-outs redrawn
- copper layers 2 -> 4
