File: modules/cellular-modem/cellular-modem.kicad_sch (KiCad schematic)
At the start: 23 parts, among them J1 MM60-mini-PCIe, J2 MM60-EZH059-B5-R650, U1 TXV0108RGYR, U2 TXV0108RGYR, U3 TXV0108RGYR, U4 TPS631000DRLR, U5 TPS631000DRLR

Commit message: Updating PART NOs
Parts:
- C1, C3: Mfr. PN (none) -> GRM219R60J476ME44D; Mouser (none) -> https://eu.mouser.com/ProductDetail/Murata-Electronics/GRM2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; Mouser_PN (none) -> GRM219R60J476ME44
- C2, C4: Mfr. PN (none) -> C2012X7S1A156M125AC; Mouser (none) -> https://eu.mouser.com/ProductDetail/TDK/C2012X7S1A156M125AC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; Mouser_PN (none) -> 810-C2012X7S1A156M1C
- J1: Mfr. PN (none) -> MM60-52B1-G1-R850; Mouser (none) -> https://eu.mouser.com/ProductDetail/JAE-Electronics/MM60-52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; Mouser_PN (none) -> 656-MM6052B1G1R850
- J2: Mfr. PN (none) -> MM60-EZH059-B5-R650; Mouser (none) -> https://eu.mouser.com/ProductDetail/JAE-Electronics/MM60-EZ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; Mouser_PN (none) -> 656-MM60-EZH059-B5-R
- JP1, JP2, M1: now left out of the parts list
- L1, L2: Mfr. PN (none) -> DFE252012P-1R0M=P2; Mouser (none) -> https://eu.mouser.com/ProductDetail/Murata-Electronics/DFE2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; Mouser_PN (none) -> 81-DFE252012P-1R0MP2
- R1, R2, R5, R6: Mfr. PN (none) -> CR0805-JW-514ELF; Mfr. PN2 (none) -> CR10514J; Mouser (none) -> https://eu.mouser.com/ProductDetail/Bourns/CR0805-JW-514ELF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; Mouser_PN (none) -> CR0805-JW-514ELF
- R3, R7: Mfr. PN (none) -> RE0805FRE0790K9L; Mouser (none) -> https://eu.mouser.com/ProductDetail/YAGEO/RE0805FRE0790K9L?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; Mouser_PN (none) -> 603-RE0805FRE0790K9L
- R8: Mfr. PN (none) -> RC0805FR-07432KL; Mouser (none) -> https://eu.mouser.com/ProductDetail/YAGEO/RC0805FR-07432KL?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; Mouser_PN (none) -> 603-RC0805FR-07432KL
- U1, U2, U3: Mfr. PN (none) -> TXV0108RGYR; Mouser (none) -> https://eu.mouser.com/ProductDetail/Texas-Instruments/TXV01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; Mouser_PN (none) -> 595-TXV0108RGYR
- U4, U5: Mfr. PN (none) -> TPS631000DRLR; Mouser (none) -> https://eu.mouser.com/ProductDetail/Texas-Instruments/TPS63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; Mouser_PN (none) -> 595-TPS631000DRLR

Commit message: Updating cellular modem - adding KiCad git ignore
Parts:
- J2: footprint MM60-EZH059-B5-R650:JAE_MM60-EZH059-B5-R650 -> cellular-modem:JAE_MM60-EZH059-B5-R650
- M1: footprint MegaCastle:MegaCastle2x28-Module-I36.0x66.3-MB00007FFFFFFFF-NIBBLE -> MegaCastle:MegaCastle2x28-Module-I42.8x66.3-MB00007FFFFFFFF-SPAREPAD; symbol MegaCastle:MegaCastle2x28-Module-I36.0x66.3-MB00007FFFFFFFF-NOCUTOUT -> MegaCastle:MegaCastle2x28-I42.8x66.3-MB00007FFFFFFFF-NOCUTOUT; now in the parts list
- U1, U2, U3: footprint VQFN24_RGY_TEX -> cellular-modem:VQFN24_RGY_TEX
- U4, U5: footprint SOT50P160X60-8N -> cellular-modem:SOT50P160X60-8N
Other:
- moved on the sheet: J1, J2, M1
