File: modules/sim-and-sd-card/sim-and-sd-card.kicad_sch (KiCad schematic)
At the start: 2 parts

Commit message: KiCad v9 adding new footprints
Parts:
- M1: footprint MegaCastle:MegaCastle2x10-Module-I16.0x20.6-MBFFFF-PANEL-NIBBLE -> MegaCastle:MegaCastle2x10-Module-I22.0x20.6-MBFFFF-SPAREPAD
Changed lines of the file:
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@@
 (kicad_sch
-	(version 20231120)
+	(version 20250114)
 	(generator "eeschema")
-	(generator_version "8.0")
+	(generator_version "9.0")
 	(paper "A4")
 	(junction
@@
 			)
 		)
-		(property "Footprint" "MegaCastle:MegaCastle2x10-Module-I16.0x20.6-MBFFFF-PANEL-NIBBLE"
+		(property "Footprint" "MegaCastle:MegaCastle2x10-Module-I22.0x20.6-MBFFFF-SPAREPAD"
 			(at 124.46 74.93 0)
 			(effects
@@
 		)
 	)
+	(embedded_fonts no)
 )
