File: modules/mems-microphone/mems-microphone.kicad_sch (KiCad schematic)
At the start: 6 parts

Commit message: Adding more mouser parts to schematics
Parts:
- C1: Mfr. PN (none) -> 12066D104KAT4A; Mouser (none) -> https://eu.mouser.com/ProductDetail/KYOCERA-AVX/12066D104KA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; Mouser PN (none) -> 581-12066D104KAT4A
- MK1: Mfr. PN (none) -> IM69D130V01XTSA1; Mouser (none) -> https://eu.mouser.com/ProductDetail/Infineon-Technologies/I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; Mouser PN (none) -> 726-IM69D130V01XTSA1
- R1, R2: Mfr. PN (none) -> AC0603JR-07100RL; Mouser (none) -> https://eu.mouser.com/ProductDetail/YAGEO/AC0603JR-07100RL?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; Mouser PN (none) -> 603-AC0603JR-07100RL
- R3: Mfr. PN (none) -> AC0603JR-07100KL; Mouser (none) -> https://eu.mouser.com/ProductDetail/YAGEO/AC0603JR-07100KL?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; Mouser PN (none) -> 603-AC0603JR-07100KL
Changed lines of the file:
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@@
+			)
+		)
+		(property "Mouser" "https://eu.mouser.com/ProductDetail/KYOCERA-AVX/12066D104KAT4A?qs=np9tehfYv7O1LpY%2FkoBbBg%3D%3D"
+			(at 50.8 55.88 0)
+			(effects
+				(font
+					(size 1.27 1.27)
+				)
+				(hide yes)
+			)
+		)
+		(property "Mouser PN" " 581-12066D104KAT4A"
+			(at 50.8 55.88 0)
+			(effects
+				(font
+					(size 1.27 1.27)
+				)
+				(hide yes)
+			)
+		)
+		(property "Mfr. PN" " 12066D104KAT4A"
+			(at 50.8 55.88 0)
+			(effects
+				(font
+					(size 1.27 1.27)
+				)
+				(hide yes)
 			)
 		)
@@
 			)
 		)
+		(property "Mouser" "https://eu.mouser.com/ProductDetail/YAGEO/AC0603JR-07100RL?qs=ygRr%2FtkhtetP1ztKDq36TA%3D%3D"
+			(at 91.44 60.96 90)
+			(effects
+				(font
+					(size 1.27 1.27)
+				)
+				(hide yes)
+			)
+		)
+		(property "Mouser PN" "603-AC0603JR-07100RL"
+			(at 91.44 60.96 90)
+			(effects
+				(font
+					(size 1.27 1.27)
+				)
+				(hide yes)
+			)
+		)
+		(property "Mfr. PN" "AC0603JR-07100RL"
+			(at 91.44 60.96 90)
+			(effects
+				(font
+					(size 1.27 1.27)
+				)
+				(hide yes)
+			)
+		)
 		(pin "2"
 		)
@@
 			)
 		)
+		(property "Mouser" "https://eu.mouser.com/ProductDetail/Infineon-Technologies/IM69D130V01XTSA1?qs=W0yvOO0ixfHjr98Yrg6FIA%3D%3D"
+			(at 77.47 60.96 0)
+			(effects
+				(font
+					(size 1.27 1.27)
+				)
+				(hide yes)
+			)
+		)
+		(property "Mouser PN" "726-IM69D130V01XTSA1"
+			(at 77.47 60.96 0)
+			(effects
+				(font
+					(size 1.27 1.27)
+				)
+				(hide yes)
+			)
+		)
+		(property "Mfr. PN" "IM69D130V01XTSA1"
+			(at 77.47 60.96 0)
+			(effects
+				(font
+					(size 1.27 1.27)
+				)
+				(hide yes)
+			)
+		)
 		(pin "4"
 		)
@@
 			)
 		)
+		(property "Mouser" "https://eu.mouser.com/ProductDetail/YAGEO/AC0603JR-07100KL?qs=cGU37fGUGy%252BuVeV1ZRovkw%3D%3D"
+			(at 87.63 49.53 0)
+			(effects
+				(font
+					(size 1.27 1.27)
+				)
+				(hide yes)
+			)
+		)
+		(property "Mouser PN" "603-AC0603JR-07100KL"
+			(at 87.63 49.53 0)
+			(effects
+				(font
+					(size 1.27 1.27)
+				)
+				(hide yes)
+			)
+		)
+		(property "Mfr. PN" "AC0603JR-07100KL"
+			(at 87.63 49.53 0)
+			(effects
+				(font
+					(size 1.27 1.27)
+				)
+				(hide yes)
+			)
+		)
 		(pin "2"
 		)
@@
 			(at 91.44 71.12 0)
 			(effects
+				(font
+					(size 1.27 1.27)
+				)
+				(hide yes)
+			)
+		)
+		(property "Mfr. PN" "AC0603JR-07100RL"
+			(at 91.44 71.12 0)
+			(effects
+				(font
+					(size 1.27 1.27)
+				)
+				(hide yes)
+			)
+		)
+		(property "Mouser" "https://eu.mouser.com/ProductDetail/YAGEO/AC0603JR-07100RL?qs=ygRr%2FtkhtetP1ztKDq36TA%3D%3D"
+			(at 91.44 71.12 0)
+			(effects
+				(font
+					(size 1.27 1.27)
+				)
+				(hide yes)
+			)
+		)
+		(property "Mouser PN" "603-AC0603JR-07100RL"
+			(at 91.44 71.12 0)
+			(effects

Commit message: Updating mems mic
Parts:
- M1: footprint MegaCastle:MegaCastle2x5-Module-I6.4x7.9-M9C4 -> MegaCastle:MegaCastle2x5-Module-I10.0x7.9-M9C4-SPAREPAD
Changed lines of the file:
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@@
 (kicad_sch
-	(version 20231120)
+	(version 20250114)
 	(generator "eeschema")
-	(generator_version "8.0")
+	(generator_version "9.0")
 	(paper "A4")
 	(junction
@@
 			)
 		)
-		(property "Footprint" "MegaCastle:MegaCastle2x5-Module-I6.4x7.9-M9C4"
+		(property "Footprint" "MegaCastle:MegaCastle2x5-Module-I10.0x7.9-M9C4-SPAREPAD"
 			(at 80.01 104.14 0)
 			(effects
@@
 		)
 	)
+	(embedded_fonts no)
 )
