File: modules/solar-and-dc-connectors/solar-and-dc-connectors.kicad_sch (KiCad schematic)
At the start: 3 parts, among them J1 S2B-PH-K-SLFSN, J2 54-00127

Commit message: Adding more mouser parts to schematics
Parts:
- J1: Mfr. PN (none) -> S2B-PH-K-S(LF)(SN); Mouser (none) -> https://eu.mouser.com/ProductDetail/JST-Commercial/S2B-PH-K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; Mouser PN (none) -> 306-S2BPHKSLFSNPP
- J2: Digikey (none) -> https://www.digikey.com/en/products/detail/tensility-intern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
Changed lines of the file:
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@@
 			)
 		)
-		(property "Datasheet" "S2B-PH-K-SLFSN"
+		(property "Datasheet" "https://eu.mouser.com/datasheet/2/564/ePH-3433490.pdf"
 			(at 102.87 46.99 0)
 			(effects
@@
 		)
 		(property "Description" ""
+			(at 102.87 46.99 0)
+			(effects
+				(font
+					(size 1.27 1.27)
+				)
+				(hide yes)
+			)
+		)
+		(property "Mouser" "https://eu.mouser.com/ProductDetail/JST-Commercial/S2B-PH-K-SLFSN?qs=cdbOS8ANM9A5Ie4gXeMjTA%3D%3D"
+			(at 102.87 46.99 0)
+			(effects
+				(font
+					(size 1.27 1.27)
+				)
+				(hide yes)
+			)
+		)
+		(property "Mouser PN" "306-S2BPHKSLFSNPP"
+			(at 102.87 46.99 0)
+			(effects
+				(font
+					(size 1.27 1.27)
+				)
+				(hide yes)
+			)
+		)
+		(property "Mfr. PN" " S2B-PH-K-S(LF)(SN) "
 			(at 102.87 46.99 0)
 			(effects
@@
 			)
 		)
-		(property "Datasheet" ""
+		(property "Datasheet" "https://tensility.s3.us-west-2.amazonaws.com/uploads/pdffiles/54-00127.pdf"
 			(at 111.76 72.39 0)
 			(effects
@@
 				(hide yes)
 			)
+		)
+		(property "Digikey" "https://www.digikey.com/en/products/detail/tensility-international-corp/54-00127/9685436"
+			(at 111.76 72.39 0)
+			(effects
+				(font
+					(size 1.27 1.27)
+				)
+				(hide yes)
+			)

Commit message: Updating solar-and-dc
Parts:
- J1: footprint CONN_S2B-PH-K-S_JST -> MegaCastle:CONN_S2B-PH-K-S_JST
- J2: footprint TENSILITY_54-00127 -> MegaCastle:TENSILITY_54-00127
- M1: footprint MegaCastle:MegaCastle2x12-Module-I12.5x25.7-M80181F -> MegaCastle:MegaCastle2x12-Module-I20.0x25.7-M80181F-SPAREPAD
Changed lines of the file:
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@@
 (kicad_sch
-	(version 20231120)
+	(version 20250114)
 	(generator "eeschema")
-	(generator_version "8.0")
+	(generator_version "9.0")
 	(paper "A4")
 	(no_connect
@@
 			)
 		)
-		(property "Footprint" "MegaCastle:MegaCastle2x12-Module-I12.5x25.7-M80181F"
+		(property "Footprint" "MegaCastle:MegaCastle2x12-Module-I20.0x25.7-M80181F-SPAREPAD"
 			(at 59.69 82.55 0)
 			(effects
@@
 			)
 		)
-		(property "Footprint" "CONN_S2B-PH-K-S_JST"
+		(property "Footprint" "MegaCastle:CONN_S2B-PH-K-S_JST"
 			(at 102.87 46.99 0)
 			(effects
@@
 			)
 		)
-		(property "Footprint" "TENSILITY_54-00127"
+		(property "Footprint" "MegaCastle:TENSILITY_54-00127"
 			(at 111.76 72.39 0)
 			(effects
@@
 		)
 	)
+	(embedded_fonts no)
 )
