File: modules/usb-c-power-in/usb-c-power-in.kicad_sch (KiCad schematic)
At the start: 2 parts, among them J1 Conn_01x02

Commit message: Updating USB-Power-IN
Parts:
- M1: footprint MegaCastle:MegaCastle2x13-Module-I14.0x28.2-M800C00C-PANEL-NIBBLE -> MegaCastle:MegaCastle2x13-Module-I20.0x28.2-M800C00C-SPAREPAD
Changed lines of the file:
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@@
 (kicad_sch
-	(version 20231120)
+	(version 20250114)
 	(generator "eeschema")
-	(generator_version "8.0")
+	(generator_version "9.0")
 	(paper "A4")
-	(no_connect
-		(at 54.61 83.82)
-	)
-	(no_connect
-		(at 40.64 55.88)
-	)
-	(no_connect
-		(at 54.61 55.88)
-	)
 	(text "These USB-C Power Delivery modules that are available on AliExpress, \nAmazon and lots of other places are pretty good, but more variable than\nthe share-price of snake oil.\n\nWATCH ESPECIALLY FOR POLARITY SWITCHING OF THE POWER OUTPUT PINS!\n\nYou shouldn't need to change anything on this schematic, as it really\nis just connecting the power and GND pins. To support other variants\nyou will instead need to go to the PCB layout, and select the footprint\nthere and then press E, and then select \"open in footprint editor\" to\nmunge it to suit your module."
 		(exclude_from_sim no)
@@
 			(justify left)
 		)
+	)
+	(no_connect
+		(at 54.61 83.82)
+	)
+	(no_connect
+		(at 40.64 55.88)
+	)
+	(no_connect
+		(at 54.61 55.88)
 	)
 	(global_label "GND"
@@
 			)
 		)
-		(property "Footprint" "MegaCastle:MegaCastle2x13-Module-I14.0x28.2-M800C00C-PANEL-NIBBLE"
+		(property "Footprint" "MegaCastle:MegaCastle2x13-Module-I20.0x28.2-M800C00C-SPAREPAD"
 			(at 46.99 93.98 0)
 			(effects
@@
 		)
 	)
+	(embedded_fonts no)
 )
