File: modules/input-power-selector/input-power-selector.kicad_sch (KiCad schematic)
At the start: 37 parts, among them Q1 SI4909DY-T1-GE3, Q2 SI4909DY-T1-GE3, Q3 SI4909DY-T1-GE3, Q4 IPF067N20NM6ATMA1, Q7 BC847, U1 LTC4417IGN, U2 SQJQ141EL-T1_GE3

Commit message: add missing footprints and symbols
Parts:
- M2: footprint MegaCastle:MegaCastle2x24-Module-I42.0x56.2-M88887D8C0001 -> MegaCastle:MegaCastle2x24-Module-I42.0x56.2-M88887D8C0001-NIBBLE
Changed lines of the file:
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@@
 			)
 		)
-		(property "Footprint" "MegaCastle:MegaCastle2x24-Module-I42.0x56.2-M88887D8C0001"
+		(property "Footprint" "MegaCastle:MegaCastle2x24-Module-I42.0x56.2-M88887D8C0001-NIBBLE"
 			(at 243.84 106.68 0)
 			(effects

Commit message: Adding Mouser parts to power selector
Parts:
- C2, C3, C5, C6, C7, C8: Manufacturer_Part_Number (none) -> 0805DC104MAT2A; Mouser (none) -> https://hr.mouser.com/ProductDetail/KYOCERA-AVX/0805DC104MA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; Mouser Part Number (none) -> 581-0805DC104MAT2A
- CR1: Manufacturer_Part_Number (none) -> SMM4F24A-TR; Mouser (none) -> https://eu.mouser.com/ProductDetail/STMicroelectronics/SMM4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; Mouser Part Number (none) -> 511-SMM4F24A-TR
- CR2: Manufacturer_Part_Number (none) -> 652-SMCJ33A; Mouser (none) -> https://eu.mouser.com/ProductDetail/Bourns/SMCJ33A?qs=%252B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; Mouser Part Number (none) -> SMCJ33A
- D1, D2: Manufacturer_Part_Number (none) -> BZX384-C30,115; Mouser (none) -> https://eu.mouser.com/ProductDetail/Nexperia/BZX384-C30115?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; Mouser Part Number (none) -> 771-BZX384-C30115
- D3: Manufacturer_Part_Number (none) -> BZX384-C12,115; Mouser (none) -> https://eu.mouser.com/ProductDetail/Nexperia/BZX384-C12115?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; Mouser Part Number (none) -> 771-BZX384-C12115
- Q1, Q2, Q3: Manufacturer_Part_Number (none) -> SI4909DY-T1-GE3; Mouser (none) -> https://eu.mouser.com/ProductDetail/Vishay-Semiconductors/S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; Mouser Part Number (none) -> 78-SI4909DY-T1-GE3
- Q4: Mouser (none) -> https://eu.mouser.com/ProductDetail/Infineon-Technologies/I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
- Q7: Manufacturer_Part_Number (none) -> 637-BC847B; Mouser (none) -> https://eu.mouser.com/ProductDetail/Diotec-Semiconductor/BC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; Mouser Part Number (none) -> BC847B
- R1, R5, R8: Mouser (none) -> https://hr.mouser.com/ProductDetail/Vishay-Dale/TNPW0805246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
- R10: Manufacturer_Part_Number (none) -> PCF0805R-100RBI; Mouser (none) -> https://hr.mouser.com/ProductDetail/Welwyn-Components-TT-El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; Mouser Part Number (none) -> 756-PCF0805R100RBI
- R11, R12, R14: Manufacturer_Part_Number (none) -> PTN0805E2463BST1; Mouser (none) -> https://eu.mouser.com/ProductDetail/Vishay-Thin-Film/PTN080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; Mouser Part Number (none) -> 71-PTN0805E2463BST1
- R13, R3, R4, R7: Manufacturer_Part_Number (none) -> RT0805DRE0711KL; Mouser (none) -> https://hr.mouser.com/ProductDetail/YAGEO/RT0805DRE0711KL?q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; Mouser Part Number (none) -> 603-RT0805DRE0711KL
- R2, R6, R9: Manufacturer_Part_Number (none) -> RV0805FR-0751KL; Mouser (none) -> https://hr.mouser.com/ProductDetail/YAGEO/RV0805FR-0751KL?q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; Mouser Part Number (none) -> 603-RV0805FR-0751KL
- U1: Manufacturer_Part_Number (none) -> LTC4417IGN#PBF; Mouser (none) -> https://eu.mouser.com/ProductDetail/Analog-Devices/LTC4417I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; Mouser Part Number (none) -> 584-LTC4417IGN#PBF
- U2: Manufacturer_Part_Number (none) -> SQJQ141EL-T1_GE3; Mouser (none) -> https://eu.mouser.com/ProductDetail/Vishay-Semiconductors/S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; Mouser Part Number (none) -> 78-SQJQ141EL-T1_GE3

Commit message: Updating footprint on input power selector
Parts:
- CR1: footprint ZDO_STMITE-FLAT_DO222-AA_STM -> (none)
- CR2: footprint DIODE_DO-214AC -> (none)
- D1, D2, D3: footprint footprints:DIO_BZX384-C30_115 -> MegaCastle:DIO_BZX384-C30_115
- M2: footprint MegaCastle:MegaCastle2x24-Module-I42.0x56.2-M88887D8C0001-NIBBLE -> MegaCastle:MegaCastle2x24-Module-I47.0x56.2-M88887D8C0001-SPAREPAD
- Q1, Q2, Q3: footprint SOIC_09DY-T1-GE3_VIS -> (none)
- Q4: footprint IPF067N20NM6ATMA1 -> (none)
- U2: footprint PowerPAK_8x8L_BWL-2_VIS -> MegaCastle:SOT95P280X120-6N
Changed lines of the file:
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@@
 (kicad_sch
-	(version 20231120)
+	(version 20250114)
 	(generator "eeschema")
-	(generator_version "8.0")
+	(generator_version "9.0")
 	(paper "A4")
+	(text "For the resistor laddars on the input power sources to\nthe source selector, we need to get V_UV and V_OV = 1V\nat the respective ends of the acceptable voltage range.\n\nIf we aim for 5V -- 28V being acceptable, then we can\nuse 246K, 51K and 11K, from VIN to GND respectively."
+		(exclude_from_sim no)
+		(at 17.78 94.742 0)
+		(effects
+			(font
+				(size 1.27 1.27)
+			)
+			(justify left)
+		)
+	)
+	(text "Filter on VOUT pin to protect against\nnegative transients if output side is shorted."
+		(exclude_from_sim no)
+		(at 141.224 184.658 0)
+		(effects
+			(font
+				(size 1.27 1.27)
+			)
+		)
+	)
+	(text "Reverse polarity protection (to 100V)\nfor Dirty DC / external solar panel."
+		(exclude_from_sim no)
+		(at 211.328 124.968 0)
+		(effects
+			(font
+				(size 1.27 1.27)
+			)
+		)
+	)
+	(text "Over-voltage protection bypass"
+		(exclude_from_sim no)
+		(at 33.528 159.004 0)
+		(effects
+			(font
+				(size 1.27 1.27)
+			)
+		)
+	)
+	(text "Detect over-voltage condition\nusing 200V tolerant TVS to\nconduct above ~24V."
+		(exclude_from_sim no)
+		(at 30.734 131.318 0)
+		(effects
+			(font
+				(size 1.27 1.27)
+			)
+			(justify left)
+		)
+	)
+	(text "Polarity protection bypass"
+		(exclude_from_sim no)
+		(at 189.738 162.814 0)
+		(effects
+			(font
+				(size 1.27 1.27)
+			)
+		)
+	)
 	(junction
 		(at 66.04 170.18)
@@
 		)
 	)
-	(text "For the resistor laddars on the input power sources to\nthe source selector, we need to get V_UV and V_OV = 1V\nat the respective ends of the acceptable voltage range.\n\nIf we aim for 5V -- 28V being acceptable, then we can\nuse 246K, 51K and 11K, from VIN to GND respectively."
-		(exclude_from_sim no)
-		(at 17.78 94.742 0)
-		(effects
-			(font
-				(size 1.27 1.27)
-			)
-			(justify left)
-		)
-	)
-	(text "Filter on VOUT pin to protect against\nnegative transients if output side is shorted."
-		(exclude_from_sim no)
-		(at 141.224 184.658 0)
-		(effects
-			(font
-				(size 1.27 1.27)
-			)
-		)
-	)
-	(text "Reverse polarity protection (to 100V)\nfor Dirty DC / external solar panel."
-		(exclude_from_sim no)
-		(at 211.328 124.968 0)
-		(effects
-			(font
-				(size 1.27 1.27)
-			)
-		)
-	)
-	(text "Over-voltage protection bypass"
-		(exclude_from_sim no)
-		(at 33.528 159.004 0)
-		(effects
-			(font
-				(size 1.27 1.27)
-			)
-		)
-	)
-	(text "Detect over-voltage condition\nusing 200V tolerant TVS to\nconduct above ~24V."
-		(exclude_from_sim no)
-		(at 30.734 131.318 0)
-		(effects
-			(font
-				(size 1.27 1.27)
-			)
-			(justify left)
-		)
-	)
-	(text "Polarity protection bypass"
-		(exclude_from_sim no)
-		(at 189.738 162.814 0)
-		(effects
-			(font
-				(size 1.27 1.27)
-			)
-		)
-	)
 	(label "OVERVOLTAGE_SENSE_UNCLAMPED"
 		(at 72.39 130.81 0)
@@
 			)
 		)
-		(property "Footprint" "footprints:DIO_BZX384-C30_115"
+		(property "Footprint" "MegaCastle:DIO_BZX384-C30_115"
 			(at 71.12 189.23 0)
 			(effects
@@
 			)
 		)
-		(property "Footprint" "SOIC_09DY-T1-GE3_VIS"
+		(property "Footprint" ""
 			(at 142.24 101.6 0)
 			(effects
@@
 			)
 		)
-		(property "Footprint" "ZDO_STMITE-FLAT_DO222-AA_STM"
+		(property "Footprint" ""
 			(at 67.31 120.65 0)
 			(effects
@@
 			)
 		)
-		(property "Footprint" "SOIC_09DY-T1-GE3_VIS"
+		(property "Footprint" ""
 			(at 140.97 41.91 0)
 			(effects
@@
 			)
 		)
-		(property "Footprint" "SOIC_09DY-T1-GE3_VIS"
+		(property "Footprint" ""
 			(at 142.24 71.12 0)
 			(effects
@@
 			)
 		)
-		(property "Footprint" "footprints:DIO_BZX384-C30_115"
+		(property "Footprint" "MegaCastle:DIO_BZX384-C30_115"
 			(at 85.09 138.43 0)
 			(effects
@@
 			)
 		)
-		(property "Footprint" "footprints:DIO_BZX384-C30_115"
+		(property "Footprint" "MegaCastle:DIO_BZX384-C30_115"
 			(at 212.09 148.59 0)
 			(effects
@@
 			)
 		)
-		(property "Footprint" "PowerPAK_8x8L_BWL-2_VIS"
+		(property "Footprint" "MegaCastle:SOT95P280X120-6N"
 			(at 234.95 142.24 0)
 			(effects
@@
 			)
 		)
-		(property "Footprint" "MegaCastle:MegaCastle2x24-Module-I42.0x56.2-M88887D8C0001-NIBBLE"
+		(property "Footprint" "MegaCastle:MegaCastle2x24-Module-I47.0x56.2-M88887D8C0001-SPAREPAD"
 			(at 243.84 106.68 0)
 			(effects
@@
 			)
 		)
-		(property "Footprint" "DIODE_DO-214AC"
+		(property "Footprint" ""
 			(at 196.85 139.7 0)
 			(effects
@@
 			)
 		)
-		(property "Footprint" "IPF067N20NM6ATMA1"
+		(property "Footprint" ""
 			(at 62.23 265.1 0)
 			(effects
@@
 		)
 	)
+	(embedded_fonts no)
 )
