File: modules/bluetooth/bluetooth.kicad_pcb (KiCad board)
At the start: 2 copper layers, 25.8 x 32.1 mm, 2 parts, among them U1 Microchip_BM83

Commit message: Update bluetooth
Parts:
- M1: footprint MegaCastle:MegaCastle2x12-Module-I19.0x25.7-M9FFFFF-PANEL-NIBBLE -> MegaCastle:MegaCastle2x12-Module-I24.0x25.7-M9FFFFF-SPAREPAD
- moved U1 0.18 mm to (109.3, 62.5)
Connections:
- net VBAT renamed VCC_3V3
Routing:
- net RFS1: track 11.6 -> 12.6 mm
- net SCLK1: track 13.1 -> 14.0 mm
- net TEMP2: track 16.4 -> 17.1 mm
- net UART_RTS: track 5.73 -> 6.45 mm
- net DT1: track 14.7 -> 15.4 mm
- net SCL: track 5.71 -> 6.41 mm
- net GND: track 6.23 -> 6.82 mm, vias 4 -> 37
- net MFB: track 13.9 -> 14.5 mm
- net UART_TXD: track 8.69 -> 9.22 mm
- net TEMP1: track 14.2 -> 14.7 mm
Other:
- board size 25.8 x 32.1 mm -> 24 x 30.5 mm
