File: modules/bluetooth/bluetooth.kicad_sch (KiCad schematic)
At the start: 2 parts, among them U1 Microchip_BM83

Commit message: Update bluetooth
Parts:
- M1: footprint MegaCastle:MegaCastle2x12-Module-I19.0x25.7-M9FFFFF-PANEL-NIBBLE -> MegaCastle:MegaCastle2x12-Module-I24.0x25.7-M9FFFFF-SPAREPAD
Changed lines of the file:
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@@
 (kicad_sch
-	(version 20231120)
+	(version 20250114)
 	(generator "eeschema")
-	(generator_version "8.0")
+	(generator_version "9.0")
 	(paper "A4")
 	(no_connect
@@
 			)
 		)
-		(property "Footprint" "MegaCastle:MegaCastle2x12-Module-I19.0x25.7-M9FFFFF-PANEL-NIBBLE"
+		(property "Footprint" "MegaCastle:MegaCastle2x12-Module-I24.0x25.7-M9FFFFF-SPAREPAD"
 			(at 54.61 105.41 0)
 			(effects
@@
 		)
 	)
+	(embedded_fonts no)
 )
